File: tad5212-board.kicad_pcb (KiCad board)
At the start: 4 copper layers, 18.2 x 25.8 mm, 22 parts, among them J1 Conn_01x10, J2 Conn_01x10, U1 XTAD5212IRGER, U2 LP5907MFX-1.8, Y2 SIT8021AI-J4-XXS-11.1E, Y3 SIT8021AI-J4-XXS-12.288E

Commit message: redo annotations
Parts:
- renumbered C7 to C10, C8 to C11, C10 to C12, C9 to C13, C12 to C5, C5 to C6, C11 to C7, C13 to C8, C6 to C9, Y3 to Y1
Changed lines of the file:
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@@
 		(descr "Capacitor SMD 0805 (2012 Metric), square (rectangular) end terminal, IPC-7351 nominal, (Body size source: IPC-SM-782 page 76, https://www.pcb-3d.com/wordpress/wp-content/uploads/ipc-sm-782a_amendment_1_and_2.pdf, https://docs.google.com/spreadsheets/d/1BsfQQcO9C6DZCsRaXUlFlo91Tg2WpOkGARC1WS5S8t0/edit?usp=sharing)")
 		(tags "capacitor")
-		(property "Reference" "C11"
+		(property "Reference" "C7"
 			(at 2.934493 0.035355 45)
 			(layer "F.SilkS")
@@
 		(descr "Capacitor SMD 0805 (2012 Metric), square (rectangular) end terminal, IPC-7351 nominal, (Body size source: IPC-SM-782 page 76, https://www.pcb-3d.com/wordpress/wp-content/uploads/ipc-sm-782a_amendment_1_and_2.pdf, https://docs.google.com/spreadsheets/d/1BsfQQcO9C6DZCsRaXUlFlo91Tg2WpOkGARC1WS5S8t0/edit?usp=sharing), generated with kicad-footprint-generator")
 		(tags "capacitor")
-		(property "Reference" "C8"
-			(at -0.106066 -1.661701 225)
+		(property "Reference" "C11"
+			(at -0.636396 -1.626346 225)
 			(layer "F.SilkS")
 			(effects
@@
 		(descr "Capacitor SMD 0603 (1608 Metric), square (rectangular) end terminal, IPC-7351 nominal, (Body size source: IPC-SM-782 page 76, https://www.pcb-3d.com/wordpress/wp-content/uploads/ipc-sm-782a_amendment_1_and_2.pdf), generated with kicad-footprint-generator")
 		(tags "capacitor")
-		(property "Reference" "C5"
+		(property "Reference" "C6"
 			(at 0 1.65 180)
 			(layer "F.SilkS")
@@
 		(descr "Capacitor SMD 0603 (1608 Metric), square (rectangular) end terminal, IPC-7351 nominal, (Body size source: IPC-SM-782 page 76, https://www.pcb-3d.com/wordpress/wp-content/uploads/ipc-sm-782a_amendment_1_and_2.pdf)")
 		(tags "capacitor")
-		(property "Reference" "C9"
+		(property "Reference" "C13"
 			(at 2.2 0 0)
 			(layer "F.SilkS")
@@
 		(layer "F.Cu")
 		(at 146.645 81.75)
-		(property "Reference" "Y3"
+		(property "Reference" "Y1"
 			(at 0.005 -1.1 0)
 			(layer "F.SilkS")
@@
 		(descr "Capacitor SMD 0603 (1608 Metric), square (rectangular) end terminal, IPC-7351 nominal, (Body size source: IPC-SM-782 page 76, https://www.pcb-3d.com/wordpress/wp-content/uploads/ipc-sm-782a_amendment_1_and_2.pdf)")
 		(tags "capacitor")
-		(property "Reference" "C10"
+		(property "Reference" "C12"
 			(at -2.65 0 0)
 			(layer "F.SilkS")
@@
 		(descr "Capacitor SMD 0805 (2012 Metric), square (rectangular) end terminal, IPC-7351 nominal, (Body size source: IPC-SM-782 page 76, https://www.pcb-3d.com/wordpress/wp-content/uploads/ipc-sm-782a_amendment_1_and_2.pdf, https://docs.google.com/spreadsheets/d/1BsfQQcO9C6DZCsRaXUlFlo91Tg2WpOkGARC1WS5S8t0/edit?usp=sharing)")
 		(tags "capacitor")
-		(property "Reference" "C13"
+		(property "Reference" "C8"
 			(at 0.106066 -5.055813 45)
 			(layer "F.SilkS")
@@
 		(descr "Capacitor SMD 0603 (1608 Metric), square (rectangular) end terminal, IPC-7351 nominal, (Body size source: IPC-SM-782 page 76, https://www.pcb-3d.com/wordpress/wp-content/uploads/ipc-sm-782a_amendment_1_and_2.pdf)")
 		(tags "capacitor")
-		(property "Reference" "C12"
+		(property "Reference" "C5"
 			(at 0 2.1 180)
 			(layer "F.SilkS")
@@
 		(descr "Capacitor SMD 0603 (1608 Metric), square (rectangular) end terminal, IPC-7351 nominal, (Body size source: IPC-SM-782 page 76, https://www.pcb-3d.com/wordpress/wp-content/uploads/ipc-sm-782a_amendment_1_and_2.pdf), generated with kicad-footprint-generator")
 		(tags "capacitor")
-		(property "Reference" "C6"
+		(property "Reference" "C9"
 			(at -2.65165 0.035355 135)
 			(layer "F.SilkS")
@@
 		(descr "Capacitor SMD 0603 (1608 Metric), square (rectangular) end terminal, IPC-7351 nominal, (Body size source: IPC-SM-782 page 76, https://www.pcb-3d.com/wordpress/wp-content/uploads/ipc-sm-782a_amendment_1_and_2.pdf), generated with kicad-footprint-generator")
 		(tags "capacitor")
-		(property "Reference" "C7"
+		(property "Reference" "C10"
 			(at -2.368808 -0.035355 225)
 			(layer "F.SilkS")
@@
 	)
 	(segment
-		(start 143.038226 77.889912)
-		(end 144.049811 76.878327)
+		(start 142.654656 77.889912)
+		(end 142.710088 77.889912)
+		(width 0.127)
+		(layer "F.Cu")
+		(net "/SDA")
+	)
+	(segment
+		(start 144 76.6)
+		(end 144 75.192911)
 		(width 0.127)
 		(layer "F.Cu")
@@
 	)
 	(segment
-		(start 144.049811 76.878327)
+		(start 144 75.192911)
 		(end 144.049811 75.1431)
 		(width 0.127)
@@
 	)
 	(segment
-		(start 142.654656 77.889912)
-		(end 143.038226 77.889912)
+		(start 142.710088 77.889912)
+		(end 144 76.6)
 		(width 0.127)
 		(layer "F.Cu")
@@
 	)
 	(segment
-		(start 142.9 77)
-		(end 143.549685 76.350315)
+		(start 143.3 75.392785)
+		(end 143.549685 75.1431)
 		(width 0.127)
 		(layer "F.Cu")
@@
 	)
 	(segment
-		(start 143.549685 76.350315)
-		(end 143.549685 75.1431)
+		(start 143.3 76.6)
+		(end 143.3 75.392785)
+		(width 0.127)
+		(layer "F.Cu")
+		(net "/SCL")
+	)
+	(segment
+		(start 142.9 77)
+		(end 143.3 76.6)
 		(width 0.127)
 		(layer "F.Cu")
@@
 	)
 	(segment
-		(start 144.549937 75.1431)
-		(end 144.549937 76.750063)
+		(start 144.5 75.193037)
+		(end 144.5 76.75)
 		(width 0.127)
 		(layer "F.Cu")
@@
 	)
 	(segment
-		(start 139.868557 81.431443)
+		(start 139.818557 81.431443)
 		(end 137.2093 81.431443)
 		(width 0.127)
@@
 	)
 	(segment
-		(start 144.549937 76.750063)
-		(end 139.868557 81.431443)
+		(start 144.549937 75.1431)
+		(end 144.5 75.193037)
 		(width 0.127)
 		(layer "F.Cu")
@@
 	)
 	(segment
-		(start 145.050063 75.1431)
-		(end 145.050063 76.699937)
+		(start 144.5 76.75)
+		(end 139.818557 81.431443)
 		(width 0.127)
 		(layer "F.Cu")
-		(net "/GPIO2")
+		(net "/GPIO1")
 	)
 	(segment
@@
 	)
 	(segment
-		(start 145.050063 76.699937)
+		(start 145 76.75)
 		(end 137.778557 83.971443)
 		(width 0.127)
@@
 	)
 	(segment
+		(start 145 75.193163)
+		(end 145 76.75)
+		(width 0.127)
+		(layer "F.Cu")
+		(net "/GPIO2")
+	)
+	(segment
+		(start 145.050063 75.1431)
+		(end 145 75.193163)
+		(width 0.127)
+		(layer "F.Cu")
+		(net "/GPIO2")
+	)
+	(segment
 		(start 144.528249 69.371751)
 		(end 144.528249 68.074265)
@@
 	)
 	(segment
-		(start 151.848357 78.2905)
-		(end 152.4493 78.891443)
+		(start 147.2545 78.2905)
+		(end 151.848357 78.2905)
 		(width 0.127)
 		(layer "F.Cu")
@@
 	)
 	(segment
-		(start 147.2545 78.2905)
-		(end 151.848357 78.2905)
+		(start 146.3 75.392785)
+		(end 146.3 77.336)
 		(width 0.127)
 		(layer "F.Cu")
@@
 	(segment
 		(start 146.050315 75.1431)
-		(end 146.050315 77.086315)
+		(end 146.3 75.392785)
+		(width 0.127)
+		(layer "F.Cu")
+		(net "/GPI1")
+	)
+	(segment
+		(start 151.848357 78.2905)
+		(end 152.4493 78.891443)
 		(width 0.127)
 		(layer "F.Cu")
@@
 	)
 	(segment
-		(start 146.050315 77.086315)
+		(start 146.3 77.336)
 		(end 147.2545 78.2905)
 		(width 0.127)
@@
 	)
 	(segment
-		(start 144.549937 70.735993)
-		(end 151.634487 63.651443)
+		(start 151.648557 63.651443)
+		(end 152.4493 63.651443)
 		(width 0.254)
 		(layer "F.Cu")
@@
 	)
 	(segment
-		(start 151.634487 63.651443)
-		(end 152.4493 63.651443)
+		(start 144.549937 70.750063)
+		(end 151.648557 63.651443)
 		(width 0.254)
 		(layer "F.Cu")
@@
 	(segment
 		(start 144.549937 71.2569)
-		(end 144.549937 70.735993)
+		(end 144.549937 70.750063)
 		(width 0.254)
 		(layer "F.Cu")
