File: tad5212-board.kicad_sch (KiCad schematic)
At the start: 21 parts, among them J1 Conn_01x10, J2 Conn_01x10, U1 XTAD5212IRGER, U2 LP5907MFX-1.8, Y2 SIT8021AI-J4-XXS-11.1E, Y3 SIT8021AI-J4-XXS-12.288E

Commit message: redo annotations
Parts:
- renumbered C7 to C10, C8 to C11, C10 to C12, C9 to C13, C12 to C5, C5 to C6, C11 to C7, C13 to C8, C6 to C9, Y3 to Y1
Changed lines of the file:
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@@
 		(dnp no)
 		(fields_autoplaced yes)
-		(property "Reference" "#PWR024"
+		(property "Reference" "#PWR026"
 			(at 267.97 114.3 0)
 			(hide yes)
@@
 			(project "tad5212-board"
 				(path "/e4005a94-2c8d-4b85-9bd4-ebc39c689406"
-					(reference "#PWR024")
+					(reference "#PWR026")
 					(unit 1)
 				)
@@
 		(dnp no)
 		(fields_autoplaced yes)
-		(property "Reference" "#PWR020"
+		(property "Reference" "#PWR011"
 			(at 130.81 120.65 0)
 			(hide yes)
@@
 			(project "tad5212-board"
 				(path "/e4005a94-2c8d-4b85-9bd4-ebc39c689406"
-					(reference "#PWR020")
+					(reference "#PWR011")
 					(unit 1)
 				)
@@
 		(dnp no)
 		(fields_autoplaced yes)
-		(property "Reference" "#PWR013"
+		(property "Reference" "#PWR015"
 			(at 152.4 46.99 0)
 			(hide yes)
@@
 			(project "tad5212-board"
 				(path "/e4005a94-2c8d-4b85-9bd4-ebc39c689406"
-					(reference "#PWR013")
+					(reference "#PWR015")
 					(unit 1)
 				)
@@
 		(dnp no)
 		(fields_autoplaced yes)
-		(property "Reference" "#PWR026"
+		(property "Reference" "#PWR010"
 			(at 127 129.54 0)
 			(hide yes)
@@
 			(project "tad5212-board"
 				(path "/e4005a94-2c8d-4b85-9bd4-ebc39c689406"
-					(reference "#PWR026")
+					(reference "#PWR010")
 					(unit 1)
 				)
@@
 		(dnp no)
 		(fields_autoplaced yes)
-		(property "Reference" "C9"
+		(property "Reference" "C13"
 			(at 262.89 113.0362 0)
 			(show_name no)
@@
 			(project "tad5212-board"
 				(path "/e4005a94-2c8d-4b85-9bd4-ebc39c689406"
-					(reference "C9")
+					(reference "C13")
 					(unit 1)
 				)
@@
 		(dnp no)
 		(fields_autoplaced yes)
-		(property "Reference" "C11"
+		(property "Reference" "C7"
 			(at 96.52 118.1162 0)
 			(show_name no)
@@
 			(project "tad5212-board"
 				(path "/e4005a94-2c8d-4b85-9bd4-ebc39c689406"
-					(reference "C11")
+					(reference "C7")
 					(unit 1)
 				)
@@
 		(dnp no)
 		(fields_autoplaced yes)
-		(property "Reference" "#PWR023"
+		(property "Reference" "#PWR022"
 			(at 200.66 114.3 0)
 			(hide yes)
@@
 			(project "tad5212-board"
 				(path "/e4005a94-2c8d-4b85-9bd4-ebc39c689406"
-					(reference "#PWR023")
+					(reference "#PWR022")
 					(unit 1)
 				)
@@
 		(dnp no)
 		(fields_autoplaced yes)
-		(property "Reference" "#PWR018"
+		(property "Reference" "#PWR020"
 			(at 187.96 135.89 0)
 			(hide yes)
@@
 			(project "tad5212-board"
 				(path "/e4005a94-2c8d-4b85-9bd4-ebc39c689406"
-					(reference "#PWR018")
+					(reference "#PWR020")
 					(unit 1)
 				)
@@
 		(dnp no)
 		(fields_autoplaced yes)
-		(property "Reference" "#PWR025"
+		(property "Reference" "#PWR08"
 			(at 93.98 129.54 0)
 			(hide yes)
@@
 			(project "tad5212-board"
 				(path "/e4005a94-2c8d-4b85-9bd4-ebc39c689406"
-					(reference "#PWR025")
+					(reference "#PWR08")
 					(unit 1)
 				)
@@
 		(dnp no)
 		(fields_autoplaced yes)
-		(property "Reference" "#PWR09"
+		(property "Reference" "#PWR07"
 			(at 92.71 120.65 0)
 			(hide yes)
@@
 			(project "tad5212-board"
 				(path "/e4005a94-2c8d-4b85-9bd4-ebc39c689406"
-					(reference "#PWR09")
+					(reference "#PWR07")
 					(unit 1)
 				)
@@
 		(dnp no)
 		(fields_autoplaced yes)
-		(property "Reference" "#PWR015"
+		(property "Reference" "#PWR016"
 			(at 152.4 116.84 0)
 			(hide yes)
@@
 			(project "tad5212-board"
 				(path "/e4005a94-2c8d-4b85-9bd4-ebc39c689406"
-					(reference "#PWR015")
+					(reference "#PWR016")
 					(unit 1)
 				)
@@
 		(dnp no)
 		(fields_autoplaced yes)
-		(property "Reference" "#PWR014"
+		(property "Reference" "#PWR09"
 			(at 116.84 134.62 0)
 			(hide yes)
@@
 			(project "tad5212-board"
 				(path "/e4005a94-2c8d-4b85-9bd4-ebc39c689406"
-					(reference "#PWR014")
+					(reference "#PWR09")
 					(unit 1)
 				)
@@
 		(dnp no)
 		(fields_autoplaced yes)
-		(property "Reference" "C5"
+		(property "Reference" "C6"
 			(at 82.5563 91.44 90)
 			(show_name no)
@@
 			(project "tad5212-board"
 				(path "/e4005a94-2c8d-4b85-9bd4-ebc39c689406"
-					(reference "C5")
+					(reference "C6")
 					(unit 1)
 				)
@@
 		(dnp no)
 		(fields_autoplaced yes)
-		(property "Reference" "C8"
+		(property "Reference" "C11"
 			(at 157.4863 63.5 90)
 			(show_name no)
@@
 			(project "tad5212-board"
 				(path "/e4005a94-2c8d-4b85-9bd4-ebc39c689406"
-					(reference "C8")
+					(reference "C11")
 					(unit 1)
 				)
@@
 		(dnp no)
 		(fields_autoplaced yes)
-		(property "Reference" "#PWR012"
+		(property "Reference" "#PWR014"
 			(at 147.32 50.8 0)
 			(hide yes)
@@
 			(project "tad5212-board"
 				(path "/e4005a94-2c8d-4b85-9bd4-ebc39c689406"
-					(reference "#PWR012")
+					(reference "#PWR014")
 					(unit 1)
 				)
@@
 		(dnp no)
 		(fields_autoplaced yes)
-		(property "Reference" "#PWR07"
+		(property "Reference" "#PWR012"
 			(at 139.7 93.98 0)
 			(hide yes)
@@
 			(project "tad5212-board"
 				(path "/e4005a94-2c8d-4b85-9bd4-ebc39c689406"
-					(reference "#PWR07")
+					(reference "#PWR012")
 					(unit 1)
 				)
@@
 		(dnp no)
 		(fields_autoplaced yes)
-		(property "Reference" "C12"
+		(property "Reference" "C5"
 			(at 74.9363 71.12 90)
 			(show_name no)
@@
 			(project "tad5212-board"
 				(path "/e4005a94-2c8d-4b85-9bd4-ebc39c689406"
-					(reference "C12")
+					(reference "C5")
 					(unit 1)
 				)
@@
 		(dnp no)
 		(fields_autoplaced yes)
-		(property "Reference" "#PWR021"
+		(property "Reference" "#PWR023"
 			(at 220.98 116.84 0)
 			(hide yes)
@@
 			(project "tad5212-board"
 				(path "/e4005a94-2c8d-4b85-9bd4-ebc39c689406"
-					(reference "#PWR021")
+					(reference "#PWR023")
 					(unit 1)
 				)
@@
 		(dnp no)
 		(fields_autoplaced yes)
-		(property "Reference" "#PWR010"
+		(property "Reference" "#PWR019"
 			(at 182.88 67.31 0)
 			(hide yes)
@@
 			(project "tad5212-board"
 				(path "/e4005a94-2c8d-4b85-9bd4-ebc39c689406"
-					(reference "#PWR010")
+					(reference "#PWR019")
 					(unit 1)
 				)
@@
 		(dnp no)
 		(fields_autoplaced yes)
-		(property "Reference" "C10"
+		(property "Reference" "C12"
 			(at 195.58 113.0362 0)
 			(show_name no)
@@
 			(project "tad5212-board"
 				(path "/e4005a94-2c8d-4b85-9bd4-ebc39c689406"
-					(reference "C10")
+					(reference "C12")
 					(unit 1)
 				)
@@
 		(dnp no)
 		(fields_autoplaced yes)
-		(property "Reference" "#PWR08"
+		(property "Reference" "#PWR013"
 			(at 143.51 64.77 0)
 			(hide yes)
@@
 			(project "tad5212-board"
 				(path "/e4005a94-2c8d-4b85-9bd4-ebc39c689406"
-					(reference "#PWR08")
+					(reference "#PWR013")
 					(unit 1)
 				)
@@
 		(dnp no)
 		(fields_autoplaced yes)
-		(property "Reference" "#PWR017"
+		(property "Reference" "#PWR025"
 			(at 265.43 124.46 0)
 			(hide yes)
@@
 			(project "tad5212-board"
 				(path "/e4005a94-2c8d-4b85-9bd4-ebc39c689406"
-					(reference "#PWR017")
+					(reference "#PWR025")
 					(unit 1)
 				)
@@
 		(dnp no)
 		(fields_autoplaced yes)
-		(property "Reference" "C7"
+		(property "Reference" "C10"
 			(at 157.4863 46.99 90)
 			(show_name no)
@@
 			(project "tad5212-board"
 				(path "/e4005a94-2c8d-4b85-9bd4-ebc39c689406"
-					(reference "C7")
+					(reference "C10")
 					(unit 1)
 				)
@@
 		(dnp no)
 		(fields_autoplaced yes)
-		(property "Reference" "C13"
+		(property "Reference" "C8"
 			(at 129.54 118.1162 0)
 			(show_name no)
@@
 			(project "tad5212-board"
 				(path "/e4005a94-2c8d-4b85-9bd4-ebc39c689406"
-					(reference "C13")
+					(reference "C8")
 					(unit 1)
 				)
@@
 		(dnp no)
 		(fields_autoplaced yes)
-		(property "Reference" "Y3"
+		(property "Reference" "Y1"
 			(at 171.45 110.49 0)
 			(show_name no)
@@
 			(project "tad5212-board"
 				(path "/e4005a94-2c8d-4b85-9bd4-ebc39c689406"
-					(reference "Y3")
+					(reference "Y1")
 					(unit 1)
 				)
@@
 		(dnp no)
 		(fields_autoplaced yes)
-		(property "Reference" "#PWR022"
+		(property "Reference" "#PWR017"
 			(at 163.83 55.88 0)
 			(hide yes)
@@
 			(project "tad5212-board"
 				(path "/e4005a94-2c8d-4b85-9bd4-ebc39c689406"
-					(reference "#PWR022")
+					(reference "#PWR017")
 					(unit 1)
 				)
@@
 		(dnp no)
 		(fields_autoplaced yes)
-		(property "Reference" "C6"
+		(property "Reference" "C9"
 			(at 149.86 58.4262 0)
 			(show_name no)
@@
 			(project "tad5212-board"
 				(path "/e4005a94-2c8d-4b85-9bd4-ebc39c689406"
-					(reference "C6")
+					(reference "C9")
 					(unit 1)
 				)
@@
 		(dnp no)
 		(fields_autoplaced yes)
-		(property "Reference" "#PWR019"
+		(property "Reference" "#PWR021"
 			(at 198.12 124.46 0)
 			(hide yes)
@@
 			(project "tad5212-board"
 				(path "/e4005a94-2c8d-4b85-9bd4-ebc39c689406"
-					(reference "#PWR019")
+					(reference "#PWR021")
 					(unit 1)
 				)
@@
 		(dnp no)
 		(fields_autoplaced yes)
-		(property "Reference" "#PWR011"
+		(property "Reference" "#PWR018"
 			(at 182.88 59.69 0)
 			(hide yes)
@@
 			(project "tad5212-board"
 				(path "/e4005a94-2c8d-4b85-9bd4-ebc39c689406"
-					(reference "#PWR011")
+					(reference "#PWR018")
 					(unit 1)
 				)
@@
 		(dnp no)
 		(fields_autoplaced yes)
-		(property "Reference" "#PWR016"
+		(property "Reference" "#PWR024"
 			(at 255.27 135.89 0)
 			(hide yes)
@@
 			(project "tad5212-board"
 				(path "/e4005a94-2c8d-4b85-9bd4-ebc39c689406"
-					(reference "#PWR016")
+					(reference "#PWR024")
 					(unit 1)
 				)
